File: led-stick.kicad_pcb (KiCad board)
At the start: 2 copper layers, 16.5 x 7 mm, 3 parts

Commit message: ready for first fab
Parts:
- added REF**: , Wire_Pads:SolderWirePad_2x_0-8mmDrill, F.Cu at (126.5, 103.0)
Routing:
- net GND: track 4.10 -> 3.23 mm
Other:
- net class Default: trace_width 0.25 -> 1.5
- net class high: trace_width 1 -> 1.5
- board text added: "+"
- board text added: "-"
Changed lines of the file:
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@@
 (kicad_pcb (version 4) (host pcbnew 4.0.5)
   (general
-    (links 11)
+    (links 13)
     (no_connects 0)
-    (area 0 0 0 0)
+    (area 121.715 99.2 142.875 106.9)
     (thickness 1.6)
-    (drawings 6)
-    (tracks 18)
+    (drawings 12)
+    (tracks 21)
     (zones 0)
-    (modules 3)
+    (modules 4)
     (nets 4)
   )
@@
   )
   (setup
-    (last_trace_width 0.25)
+    (last_trace_width 1.5)
     (trace_clearance 0.2)
     (zone_clearance 0.508)
@@
     (mod_text_size 1 1)
     (mod_text_width 0.15)
-    (pad_size 1.524 1.524)
-    (pad_drill 0.762)
+    (pad_size 1.99898 1.99898)
+    (pad_drill 0.8001)
     (pad_to_mask_clearance 0.2)
     (aux_axis_origin 0 0)
     (grid_origin 117.5 93.5)
-    (visible_elements FFFFFF7F)
+    (visible_elements 7FFFFFFF)
     (pcbplotparams
-      (layerselection 0x00030_80000001)
+      (layerselection 0x31cf0_80000001)
       (usegerberextensions false)
       (excludeedgelayer true)
@@
       (outputformat 1)
       (mirror false)
-      (drillshape 1)
+      (drillshape 0)
       (scaleselection 1)
-      (outputdirectory ""))
+      (outputdirectory gerber/))
   )
   (net 0 "")
@@
   (net_class Default "This is the default net class."
     (clearance 0.2)
-    (trace_width 0.25)
+    (trace_width 1.5)
     (via_dia 0.6)
     (via_drill 0.4)
@@
   (net_class high ""
     (clearance 0.2)
-    (trace_width 1)
+    (trace_width 1.5)
     (via_dia 1.5)
     (via_drill 1)
@@
     )
   )
+  (module Wire_Pads:SolderWirePad_2x_0-8mmDrill (layer F.Cu)
+    (at 126.5 103 90)
+    (fp_text reference REF** (at 0 -3.81 90) (layer F.SilkS) hide
+      (effects (font (size 1 1) (thickness 0.15)))
+    )
+    (fp_text value "" (at 0.635 2.54 90) (layer F.Fab) hide
+      (effects (font (size 1 1) (thickness 0.15)))
+    )
+    (pad 1 thru_hole circle (at -1.905 0 90) (size 1.99898 1.99898) (drill 0.8001) (layers *.Cu *.Mask)
+      (net 2 VCC))
+    (pad 2 thru_hole circle (at 1.905 0 90) (size 1.99898 1.99898) (drill 0.8001) (layers *.Cu *.Mask)
+      (net 3 GND))
+  )
+  (gr_text - (at 136.5 106) (layer B.SilkS)
+    (effects (font (size 1 1) (thickness 0.2)) (justify mirror))
+  )
+  (gr_text + (at 136.5 100) (layer B.SilkS)
+    (effects (font (size 1 1) (thickness 0.2)) (justify mirror))
+  )
+  (gr_text - (at 128.5 101) (layer B.SilkS)
+    (effects (font (size 1.5 1.5) (thickness 0.3)) (justify mirror))
+  )
+  (gr_text + (at 128.5 105) (layer B.SilkS)
+    (effects (font (size 1.5 1.5) (thickness 0.3)) (justify mirror))
+  )
+  (gr_text - (at 125.5 102) (layer F.SilkS)
+    (effects (font (size 0.5 0.5) (thickness 0.125)))
+  )
+  (gr_text + (at 125.5 104) (layer F.SilkS)
+    (effects (font (size 0.5 0.5) (thickness 0.125)))
+  )
   (gr_line (start 125 106.5) (end 125.5 106.5) (angle 90) (layer Edge.Cuts) (width 0.15))
   (gr_line (start 125 99.5) (end 125 106.5) (angle 90) (layer Edge.Cuts) (width 0.15))
@@
   (gr_line (start 141.5 99.5) (end 141.5 106.5) (angle 90) (layer Edge.Cuts) (width 0.15))
   (gr_line (start 125.5 99.5) (end 141.5 99.5) (angle 90) (layer Edge.Cuts) (width 0.15))
-  (segment (start 135.1 104.55) (end 134 104.55) (width 1) (layer F.Cu) (net 1) (status C00000))
-  (segment (start 134 104.55) (end 132.9 104.55) (width 1) (layer F.Cu) (net 1) (status C00000))
-  (segment (start 132.9 104.55) (end 132 105.45) (width 1) (layer F.Cu) (net 1) (status 400000))
-  (segment (start 132 105.45) (end 129.5 105.45) (width 1) (layer F.Cu) (net 1) (status 800000))
-  (segment (start 140.1 104.55) (end 139 104.55) (width 1) (layer F.Cu) (net 1) (status C00000))
-  (segment (start 139 104.55) (end 137.9 104.55) (width 1) (layer F.Cu) (net 1) (status C00000))
-  (segment (start 137.9 104.55) (end 135.1 104.55) (width 1) (layer F.Cu) (net 1) (status C00000))
-  (segment (start 132.9 101.45) (end 132.55 101.45) (width 1) (layer F.Cu) (net 2) (status C00000))
-  (segment (start 132.55 101.45) (end 131 103) (width 1) (layer F.Cu) (net 2) (status 400000))
-  (segment (start 127.5 103) (end 126 104.5) (width 1) (layer F.Cu) (net 2))
-  (segment (start 131 103) (end 127.5 103) (width 1) (layer F.Cu) (net 2))
-  (segment (start 140.1 101.45) (end 139 101.45) (width 1) (layer F.Cu) (net 2) (status C00000))
-  (segment (start 139 101.45) (end 137.9 101.45) (width 1) (layer F.Cu) (net 2) (status C00000))
-  (segment (start 137.9 101.45) (end 135.1 101.45) (width 1) (layer F.Cu) (net 2) (status C00000))
-  (segment (start 135.1 101.45) (end 134 101.45) (width 1) (layer F.Cu) (net 2) (status C00000))
-  (segment (start 134 101.45) (end 132.9 101.45) (width 1) (layer F.Cu) (net 2) (status C00000))
-  (segment (start 129.5 100.55) (end 127.45 100.55) (width 1) (layer F.Cu) (net 3) (status 400000))
-  (segment (start 127.45 100.55) (end 126 102) (width 1) (layer F.Cu) (net 3))
+  (segment (start 132.9 104.55) (end 132.45 104.55) (width 1.5) (layer F.Cu) (net 1) (status 400000))
+  (segment (start 131.55 105.45) (end 129.5 105.45) (width 1.5) (layer F.Cu) (net 1) (status 800000))
+  (segment (start 132.45 104.55) (end 131.55 105.45) (width 1.5) (layer F.Cu) (net 1))
+  (segment (start 134 104.55) (end 132.9 104.55) (width 1.5) (layer F.Cu) (net 1) (status C00000))
+  (segment (start 135.1 104.55) (end 134 104.55) (width 1.5) (layer F.Cu) (net 1) (status C00000))
+  (segment (start 137.9 104.55) (end 135.1 104.55) (width 1.5) (layer F.Cu) (net 1) (status C00000))
+  (segment (start 139 104.55) (end 137.9 104.55) (width 1.5) (layer F.Cu) (net 1) (status C00000))
+  (segment (start 140.1 104.55) (end 139 104.55) (width 1.5) (layer F.Cu) (net 1) (status C00000))
+  (segment (start 139 101.45) (end 140.1 101.45) (width 1.5) (layer F.Cu) (net 2) (status C00000))
+  (segment (start 137.9 101.45) (end 139 101.45) (width 1.5) (layer F.Cu) (net 2) (status C00000))
+  (segment (start 135.1 101.45) (end 137.9 101.45) (width 1.5) (layer F.Cu) (net 2) (status C00000))
+  (segment (start 134 101.45) (end 135.1 101.45) (width 1.5) (layer F.Cu) (net 2) (status C00000))
+  (segment (start 132.9 101.45) (end 134 101.45) (width 1.5) (layer F.Cu) (net 2) (status C00000))
+  (segment (start 132.9 101.45) (end 132.05 101.45) (width 1.5) (layer F.Cu) (net 2) (status 400000))
+  (segment (start 130 103.5) (end 131.5 102) (width 1.5) (layer F.Cu) (net 2))
+  (segment (start 127 103.5) (end 130 103.5) (width 1.5) (layer F.Cu) (net 2))
+  (segment (start 127 103.5) (end 126.5 104) (width 1.5) (layer F.Cu) (net 2))
+  (segment (start 132.05 101.45) (end 131.5 102) (width 1.5) (layer F.Cu) (net 2))
+  (segment (start 126.5 104.905) (end 126.5 104) (width 1.5) (layer F.Cu) (net 2))
+  (segment (start 126.5 101.095) (end 128.955 101.095) (width 1.5) (layer F.Cu) (net 3))
+  (segment (start 128.955 101.095) (end 129.5 100.55) (width 1.5) (layer F.Cu) (net 3))
 )
